File: variants/battery-kit/hardware/kicad/MistMaker-Battery-Kit-V0-3.kicad_sch (KiCad schematic)
At the start: 70 parts, among them IC1 TPS61023, IC2 TPS2116DRLR, J1 Conn_01x07_Socket, J10 Conn_01x07_Socket, J11 Conn_01x01, J12 Conn_01x01, J13 Conn_01x01, J14 Conn_01x01, J15 Conn_01x01, J2 PH-2PWB, J3 PH-2PWB, J4 Conn_01x01, J5 Conn_01x01, J6 Qwiic_Vertical, J7 Conn_01x07_Socket, J8 Conn_01x07_Socket, J9 Conn_01x01, Q1 2N7002, Q4 DMT10H009LCG-7, U1 LP4060B5F, U2 AP7361C-3.3V, U3 INA180A3, U4 UCC27511ADBV

Commit message: Battery Kit V0.3: fix bulk-cap part C25804 (10kΩ resistor) → C96446 (10µF 25V X5R)
C5/C6/C12/C15/C16 carried a 10kΩ resistor LCSC number in the 10µF
positions (charger/boost bulk caps). Netlist analysis: C5 sat directly
across BATT+ → ~0.4mA permanent battery bleed. Fixed in schematic,
PCB, and re-exported production files (synced from Drive working copy).

Co-Authored-By: Claude Fable 5 <noreply@anthropic.com>
Parts:
- C12, C15, C16, C5, C6: LCSC C25804 -> C96446
Changed lines of the file:
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@@
 			)
 		)
-		(property "LCSC" "C25804"
+		(property "LCSC" "C96446"
 			(at 102.87 58.42 0)
 			(hide yes)
@@
 			)
 		)
-		(property "LCSC" "C25804"
+		(property "LCSC" "C96446"
 			(at 189.23 52.07 0)
 			(hide yes)
@@
 			)
 		)
-		(property "LCSC" "C25804"
+		(property "LCSC" "C96446"
 			(at 229.87 52.07 0)
 			(hide yes)
@@
 			)
 		)
-		(property "LCSC" "C25804"
+		(property "LCSC" "C96446"
 			(at 92.71 52.07 0)
 			(hide yes)
@@
 			)
 		)
-		(property "LCSC" "C25804"
+		(property "LCSC" "C96446"
 			(at 170.18 58.42 0)
 			(hide yes)

Commit message: Relink schematic to reorganized kicad-libraries buckets
3 symbol refs + 2 footprint fields repointed to the new central library:
  DavidLib_Mux:TPS2116DRLR        -> DavidLib_Power:TPS2116DRLR
  DavidLib_Switch:N_MOSFET_G1003A -> DavidLib_Discrete:N_MOSFET_G1003A
  Switch_DavidLib:TS-1088-AR02016 -> DavidLib_Switch:TS-1088-AR02016 (also fixes a typo'd nickname)
  + matching Footprint fields (TPS62932DRLR, TS1088AR02016)

Verified: all refs resolve against the new repo; kicad-cli ERC loads clean
(24 violations, same as before). Original kept as .bak-20260623-115400.

Co-Authored-By: Claude Opus 4.8 (1M context) <noreply@anthropic.com>
Parts:
- IC2: footprint DavidLib_Mux:TPS62932DRLR -> DavidLib_Power:TPS62932DRLR; symbol DavidLib_Mux:TPS2116DRLR -> DavidLib_Power:TPS2116DRLR
- Q4: symbol DavidLib_Switch:N_MOSFET_G1003A -> DavidLib_Discrete:N_MOSFET_G1003A
- S2: symbol Switch_DavidLib:TS-1088-AR02016 -> DavidLib_Switch:TS-1088-AR02016
Changed lines of the file:
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@@
 	)
 	(symbol
-		(lib_id "DavidLib_Mux:TPS2116DRLR")
+		(lib_id "DavidLib_Power:TPS2116DRLR")
 		(at 116.84 36.83 0)
 		(unit 1)
@@
 			)
 		)
-		(property "Footprint" "DavidLib_Mux:TPS62932DRLR"
+		(property "Footprint" "DavidLib_Power:TPS62932DRLR"
 			(at 146.05 131.75 0)
 			(hide yes)
@@
 	)
 	(symbol
-		(lib_id "Switch_DavidLib:TS-1088-AR02016")
+		(lib_id "DavidLib_Switch:TS-1088-AR02016")
 		(at 337.82 222.25 0)
 		(unit 1)
@@
 	)
 	(symbol
-		(lib_id "DavidLib_Switch:N_MOSFET_G1003A")
+		(lib_id "DavidLib_Discrete:N_MOSFET_G1003A")
 		(at 154.94 153.67 0)
 		(unit 1)
